File: PCB/LedDriver/digitDriver.kicad_sch (KiCad schematic)
At the start: 43 parts, among them U201 NJW4617DL3-TE1, U202 NJW4617DL3-TE1, U203 NJW4617DL3-TE1, U204 NJW4617DL3-TE1, U205 NJW4617DL3-TE1, U206 NJW4617DL3-TE1, U207 NJW4617DL3-TE1, U208 74HC595

Commit message: 基板改良
Parts:
- removed R228: 1k, Resistor_SMD:R_0603_1608Metric, symbol Device:R
- added C201, C202, C203, C204, C205, C206, C207, C208: 0.1u, Capacitor_SMD:C_0603_1608Metric, symbol Device:C
- added R222: 1.2k, Resistor_SMD:R_0603_1608Metric, symbol Device:R
- R201, R204, R207, R210, R213, R216, R219: value 680 -> 1.2k
- R202, R205, R208, R211, R214, R217, R220: value 0.33 -> 0.20; footprint Resistor_THT:R_Axial_DIN0207_L6.3mm_D2.5mm_P7.62mm_Horizontal -> Resistor_THT:R_Axial_DIN0207_L6.3mm_D2.5mm_P10.16mm_Horizontal
- R203, R206, R209, R212, R215, R218, R221: value 0.33 -> 0.47; footprint Resistor_THT:R_Axial_DIN0207_L6.3mm_D2.5mm_P7.62mm_Horizontal -> Resistor_THT:R_Axial_DIN0207_L6.3mm_D2.5mm_P10.16mm_Horizontal
- R223, R224, R225, R226, R227: value 1k -> 1.2k
- R228: renamed from R222; value 1k -> 1.2k
Connections:
- net +3.3V: now also C201.1, C202.1, C203.1, C204.1, C205.1, C206.1, C207.1, C208.2
- net GND: now also C201.2, C202.2, C203.2, C204.2, C205.2, C206.2, C207.2, C208.1, R222.2
- net QA: now also R222.1
- net QB: now also R223.1; no longer R227.1
- net QC: now also R224.1; no longer R226.1
- net QE: now also R226.1; no longer R224.1
- net QF: now also R227.1; no longer R223.1
- net at R214.1: now also U205.4 (RS); no longer R215.1
- net at R214.2: now also R215.1; no longer U205.4 (RS)
- net at U207.4 (RS): now also R220.1; no longer R220.2
- net at R211.2: now also R212.1; no longer U204.4 (RS)
- net at R206.1: now also R205.2; no longer R205.1
- net at U202.4 (RS): now also R205.1; no longer R205.2
- net at R202.2: now also R203.1; no longer U201.4 (RS)
- net at R218.1: now also R217.2; no longer R217.1
- net at U206.4 (RS): now also R217.1; no longer R217.2
- net at R209.1: now also R208.2; no longer R208.1
- net at U203.4 (RS): now also R208.1; no longer R208.2
- net at R202.1: now also U201.4 (RS); no longer R203.1
- net at R221.1: now also R220.2; no longer R220.1
- net at R211.1: now also U204.4 (RS); no longer R212.1
Other:
- moved on the sheet: D202, D203, D205, D206, D207, R204, R228, U202, U203, U205, U206, U207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

Commit message: パターン修正
LEDドライバのパスコンを最短で配線
LEDドライバのタブをGNDに配線
平行な信号パターン同士の距離を開け、GNDパターンを間に追加
直角なパターンを修正
Connections:
- net _SCLR is gone; now on net +3.3V: U208.10 (~{SRCLR})
- net GND: now also U201.6 (EP), U202.6 (EP), U203.6 (EP), U204.6 (EP), U205.6 (EP), U206.6 (EP), U207.6 (EP)
- no-connect marks 8 -> 1
Changed lines of the file:
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@@
   (junction (at 91.44 33.02) (diameter 0) (color 0 0 0 0)
   )
+  (junction (at 260.35 45.72) (diameter 0) (color 0 0 0 0)
+  )
   (junction (at 19.05 93.98) (diameter 0) (color 0 0 0 0)
   )
   (junction (at 97.79 182.88) (diameter 0) (color 0 0 0 0)
   )
+  (junction (at 53.34 106.68) (diameter 0) (color 0 0 0 0)
+  )
   (junction (at 120.65 182.88) (diameter 0) (color 0 0 0 0)
   )
+  (junction (at 124.46 106.68) (diameter 0) (color 0 0 0 0)
+  )
   (junction (at 54.61 146.05) (diameter 0) (color 0 0 0 0)
   )
   (junction (at 161.29 93.98) (diameter 0) (color 0 0 0 0)
   )
+  (junction (at 195.58 106.68) (diameter 0) (color 0 0 0 0)
+  )
   (junction (at 260.35 27.94) (diameter 0) (color 0 0 0 0)
   )
@@
   (junction (at 195.58 88.9) (diameter 0) (color 0 0 0 0)
   )
+  (junction (at 196.85 45.72) (diameter 0) (color 0 0 0 0)
+  )
   (junction (at 124.46 88.9) (diameter 0) (color 0 0 0 0)
   )
   (junction (at 90.17 182.88) (diameter 0) (color 0 0 0 0)
   )
+  (junction (at 54.61 45.72) (diameter 0) (color 0 0 0 0)
+  )
   (junction (at 53.34 88.9) (diameter 0) (color 0 0 0 0)
   )
@@
   (junction (at 54.61 27.94) (diameter 0) (color 0 0 0 0)
   )
+  (junction (at 125.73 45.72) (diameter 0) (color 0 0 0 0)
+  )
   (junction (at 105.41 182.88) (diameter 0) (color 0 0 0 0)
   )
@@
   (junction (at 162.56 33.02) (diameter 0) (color 0 0 0 0)
   )
-  (no_connect (at 53.34 43.18))
-  (no_connect (at 124.46 43.18))
-  (no_connect (at 259.08 43.18))
-  (no_connect (at 123.19 104.14))
   (no_connect (at 64.77 156.21))
-  (no_connect (at 52.07 104.14))
-  (no_connect (at 194.31 104.14))
-  (no_connect (at 195.58 43.18))
   (wire (pts (xy 54.61 146.05) (xy 54.61 151.13))
     (stroke (width 0) (type default) (color 0 0 0 0))
@@
     (stroke (width 0) (type default) (color 0 0 0 0))
   )
+  (wire (pts (xy 259.08 43.18) (xy 260.35 43.18))
+    (stroke (width 0) (type default) (color 0 0 0 0))
+  )
   (wire (pts (xy 140.97 38.1) (xy 140.97 27.94))
     (stroke (width 0) (type default) (color 0 0 0 0))
@@
     (stroke (width 0) (type default) (color 0 0 0 0))
   )
+  (wire (pts (xy 260.35 43.18) (xy 260.35 45.72))
+    (stroke (width 0) (type default) (color 0 0 0 0))
+  )
   (wire (pts (xy 73.66 182.88) (xy 81.28 182.88))
     (stroke (width 0) (type default) (color 0 0 0 0))
@@
     (stroke (width 0) (type default) (color 0 0 0 0))
   )
+  (wire (pts (xy 194.31 104.14) (xy 195.58 104.14))
+    (stroke (width 0) (type default) (color 0 0 0 0))
+  )
   (wire (pts (xy 19.05 95.25) (xy 19.05 93.98))
     (stroke (width 0) (type default) (color 0 0 0 0))
@@
     (stroke (width 0) (type default) (color 0 0 0 0))
   )
+  (wire (pts (xy 54.61 43.18) (xy 54.61 45.72))
+    (stroke (width 0) (type default) (color 0 0 0 0))
+  )
   (wire (pts (xy 68.58 119.38) (xy 68.58 106.68))
     (stroke (width 0) (type default) (color 0 0 0 0))
@@
     (stroke (width 0) (type default) (color 0 0 0 0))
   )
+  (wire (pts (xy 35.56 162.56) (xy 35.56 163.83))
+    (stroke (width 0) (type default) (color 0 0 0 0))
+  )
   (wire (pts (xy 54.61 45.72) (xy 54.61 46.99))
     (stroke (width 0) (type default) (color 0 0 0 0))
   )
+  (wire (pts (xy 53.34 43.18) (xy 54.61 43.18))
+    (stroke (width 0) (type default) (color 0 0 0 0))
+  )
   (wire (pts (xy 194.31 88.9) (xy 195.58 88.9))
     (stroke (width 0) (type default) (color 0 0 0 0))
@@
     (stroke (width 0) (type default) (color 0 0 0 0))
   )
+  (wire (pts (xy 196.85 43.18) (xy 196.85 45.72))
+    (stroke (width 0) (type default) (color 0 0 0 0))
+  )
   (wire (pts (xy 64.77 166.37) (xy 97.79 166.37))
     (stroke (width 0) (type default) (color 0 0 0 0))
   )
+  (wire (pts (xy 195.58 43.18) (xy 196.85 43.18))
+    (stroke (width 0) (type default) (color 0 0 0 0))
+  )
   (wire (pts (xy 53.34 146.05) (xy 54.61 146.05))
     (stroke (width 0) (type default) (color 0 0 0 0))
@@
     (stroke (width 0) (type default) (color 0 0 0 0))
   )
+  (wire (pts (xy 53.34 104.14) (xy 53.34 106.68))
+    (stroke (width 0) (type default) (color 0 0 0 0))
+  )
   (wire (pts (xy 194.31 99.06) (xy 199.39 99.06))
     (stroke (width 0) (type default) (color 0 0 0 0))
@@
     (stroke (width 0) (type default) (color 0 0 0 0))
   )
+  (wire (pts (xy 52.07 104.14) (xy 53.34 104.14))
+    (stroke (width 0) (type default) (color 0 0 0 0))
+  )
   (wire (pts (xy 52.07 88.9) (xy 53.34 88.9))
     (stroke (width 0) (type default) (color 0 0 0 0))
@@
     (stroke (width 0) (type default) (color 0 0 0 0))
   )
+  (wire (pts (xy 123.19 104.14) (xy 124.46 104.14))
+    (stroke (width 0) (type default) (color 0 0 0 0))
+  )
+  (wire (pts (xy 124.46 104.14) (xy 124.46 106.68))
+    (stroke (width 0) (type default) (color 0 0 0 0))
+  )
   (wire (pts (xy 140.97 58.42) (xy 140.97 45.72))
     (stroke (width 0) (type default) (color 0 0 0 0))
@@
     (stroke (width 0) (type default) (color 0 0 0 0))
   )
-  (wire (pts (xy 43.18 163.83) (xy 44.45 163.83))
+  (wire (pts (xy 35.56 163.83) (xy 44.45 163.83))
     (stroke (width 0) (type default) (color 0 0 0 0))
   )
@@
     (stroke (width 0) (type default) (color 0 0 0 0))
   )
+  (wire (pts (xy 195.58 104.14) (xy 195.58 106.68))
+    (stroke (width 0) (type default) (color 0 0 0 0))
+  )
   (wire (pts (xy 64.77 179.07) (xy 66.04 179.07))
     (stroke (width 0) (type default) (color 0 0 0 0))
   )
+  (wire (pts (xy 125.73 43.18) (xy 125.73 45.72))
+    (stroke (width 0) (type default) (color 0 0 0 0))
+  )
   (wire (pts (xy 53.34 88.9) (xy 68.58 88.9))
     (stroke (width 0) (type default) (color 0 0 0 0))
@@
   )
   (wire (pts (xy 90.17 182.88) (xy 97.79 182.88))
+    (stroke (width 0) (type default) (color 0 0 0 0))
+  )
+  (wire (pts (xy 124.46 43.18) (xy 125.73 43.18))
     (stroke (width 0) (type default) (color 0 0 0 0))
   )
@@
   (hierarchical_label "QH" (shape input) (at 66.04 179.07 0)
     (effects (font (size 1.27 1.27)) (justify left))
-  )
-  (hierarchical_label "_SCLR" (shape input) (at 43.18 163.83 180)
-    (effects (font (size 1.27 1.27)) (justify right))
   )
   (hierarchical_label "_G" (shape input) (at 43.18 171.45 180)
@@
     (pin "2")
   )
+  (symbol (lib_id "power:+3.3V") (at 35.56 162.56 0) (unit 1)
+    (in_bom yes) (on_board yes) (fields_autoplaced)
+    (property "Reference" "#PWR?" (id 0) (at 35.56 166.37 0)
+      (effects (font (size 1.27 1.27)) hide)
+    )
+    (property "Value" "+3.3V" (id 1) (at 35.56 157.48 0))
+    (property "Footprint" "" (id 2) (at 35.56 162.56 0)
+      (effects (font (size 1.27 1.27)) hide)
+    )
+    (property "Datasheet" "" (id 3) (at 35.56 162.56 0)
+      (effects (font (size 1.27 1.27)) hide)
+    )
+    (pin "1")
+  )
   (symbol (lib_id "power:+3.3V") (at 54.61 26.67 0) (unit 1)
